File: DO_AN_DKTD/STM32.kicad_sch (KiCad schematic)
At the start: 25 parts, among them J3 Conn_01x05_Male, SW2 SW_Push, U4 STM32F103C8Tx, Y1 Crystal_GND24_Small

Commit message: add testoint SPI USB LEDTEST and Buck power
Parts:
- added J11: Conn_01x03_Pin, Connector_PinHeader_2.00mm:PinHeader_1x03_P2.00mm_Vertical, symbol Connector:Conn_01x03_Pin
Connections:
- net Led_test1: now also J11.1 (Pin_1)
- net Led_test2: now also J11.2 (Pin_2)
- net Led_test3: now also J11.3 (Pin_3)

Commit message: commit to change branch
Changed lines of the file:
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@@
     (stroke (width 0) (type default))
   )
-  (bus_entry (at 323.215 226.06) (size 2.54 2.54)
+  (bus_entry (at 297.815 198.755) (size 2.54 2.54)
     (stroke (width 0) (type default))
   )
@@
     (stroke (width 0) (type default))
   )
-  (bus_entry (at 323.215 223.52) (size 2.54 2.54)
+  (bus_entry (at 297.815 196.215) (size 2.54 2.54)
     (stroke (width 0) (type default))
   )
@@
     (stroke (width 0) (type default))
   )
-  (bus_entry (at 323.215 220.98) (size 2.54 2.54)
+  (bus_entry (at 297.815 193.675) (size 2.54 2.54)
     (stroke (width 0) (type default))
   )
@@
     (stroke (width 0) (type default))
   )
-  (polyline (pts (xy 345.44 249.555) (xy 76.835 249.555))
+  (polyline (pts (xy 345.44 234.315) (xy 76.835 234.315))
     (stroke (width 0) (type default))
   )
@@
     (stroke (width 0) (type default))
   )
-  (wire (pts (xy 314.325 220.98) (xy 323.215 220.98))
+  (wire (pts (xy 288.925 193.675) (xy 297.815 193.675))
     (stroke (width 0) (type default))
   )
@@
     (stroke (width 0) (type default))
   )
-  (wire (pts (xy 314.325 226.06) (xy 323.215 226.06))
+  (wire (pts (xy 288.925 198.755) (xy 297.815 198.755))
     (stroke (width 0) (type default))
   )
@@
     (stroke (width 0) (type default))
   )
-  (polyline (pts (xy 345.44 107.315) (xy 345.44 249.555))
+  (polyline (pts (xy 345.44 107.315) (xy 345.44 234.315))
     (stroke (width 0) (type default))
   )
@@
     (stroke (width 0) (type default))
   )
-  (wire (pts (xy 314.325 223.52) (xy 323.215 223.52))
+  (wire (pts (xy 288.925 196.215) (xy 297.815 196.215))
     (stroke (width 0) (type default))
   )
@@
     (stroke (width 0) (type default))
   )
-  (polyline (pts (xy 76.835 107.315) (xy 76.835 249.555))
+  (polyline (pts (xy 76.835 107.315) (xy 76.835 234.315))
     (stroke (width 0) (type default))
   )
@@
     (stroke (width 0) (type default))
   )
-  (bus (pts (xy 325.755 226.06) (xy 325.755 228.6))
+  (bus (pts (xy 300.355 198.755) (xy 300.355 201.295))
     (stroke (width 0) (type default))
   )
@@
     (stroke (width 0) (type default))
   )
-  (bus (pts (xy 325.755 228.6) (xy 325.755 229.235))
+  (bus (pts (xy 300.355 201.295) (xy 300.355 201.93))
     (stroke (width 0) (type default))
   )
@@
     (stroke (width 0) (type default))
   )
-  (bus (pts (xy 325.755 229.235) (xy 328.295 229.235))
+  (bus (pts (xy 300.355 201.93) (xy 302.895 201.93))
     (stroke (width 0) (type default))
   )
@@
     (stroke (width 0) (type default))
   )
-  (bus (pts (xy 325.755 223.52) (xy 325.755 226.06))
+  (bus (pts (xy 300.355 196.215) (xy 300.355 198.755))
     (stroke (width 0) (type default))
   )
@@
     (stroke (width 0) (type default))
   )
-  (text "STM32F103C8T6\n" (at 170.18 244.475 0)
+  (text "STM32F103C8T6\n" (at 173.99 230.505 0)
     (effects (font (size 5 5) (thickness 1) bold) (justify left bottom))
   )
@@
     (effects (font (size 1.27 1.27)) (justify left bottom))
   )
-  (label "LORA.RST" (at 314.325 223.52 0) (fields_autoplaced)
+  (label "LORA.RST" (at 288.925 196.215 0) (fields_autoplaced)
     (effects (font (size 1.27 1.27)) (justify left bottom))
   )
@@
     (effects (font (size 1.27 1.27)) (justify left bottom))
   )
-  (label "LORA.INT" (at 314.325 220.98 0) (fields_autoplaced)
+  (label "LORA.INT" (at 288.925 193.675 0) (fields_autoplaced)
     (effects (font (size 1.27 1.27)) (justify left bottom))
   )
@@
     (effects (font (size 1.27 1.27)) (justify left bottom))
   )
-  (label "LORA.CS" (at 314.325 226.06 0) (fields_autoplaced)
+  (label "LORA.CS" (at 288.925 198.755 0) (fields_autoplaced)
     (effects (font (size 1.27 1.27)) (justify left bottom))
   )
@@
     (effects (font (size 1.27 1.27)) (justify left))
   )
-  (hierarchical_label "LORA{pLORA}" (shape input) (at 328.295 229.235 0) (fields_autoplaced)
+  (hierarchical_label "LORA{pLORA}" (shape input) (at 302.895 201.93 0) (fields_autoplaced)
     (effects (font (size 1.27 1.27)) (justify left))
   )
