File: DO_AN_DKTD/ESP.kicad_sch (KiCad schematic)
At the start: 11 parts, among them J4 , SW2 SW_Push, SW3 SW_Push, U10 ESP-07

Commit message: commit to change branch
Other:
- note added: "ESP8266"
- moved on the sheet: C35, C5, R51, U10

Commit message: config pin STM32 CubeIDE, and add resistor ESP8266
Parts:
- added R51 (x3): 10k, IVS_FOOTPRINTS:R_0603, symbol Device:R
Connections:
- net +3V3: now also R51.2, R51.2
- net BOOT: now also U10.18 (GPIO0); no longer U10.3 (EN)
- net GND: now also R51.1
- net at U10.16 (GPIO15): now also R51.2
- net at U10.17 (GPIO2): now also R51.1
- new net: R51.1, U10.3 (EN)
- no-connect marks 8 -> 5
Changed lines of the file:
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@@
   (junction (at 102.87 67.945) (diameter 0) (color 0 0 0 0)
   )
+  (junction (at 97.79 67.945) (diameter 0) (color 0 0 0 0)
+  )
   (junction (at 185.42 136.525) (diameter 0) (color 0 0 0 0)
   )
@@
   (junction (at 185.42 100.965) (diameter 0) (color 0 0 0 0)
   )
-  (no_connect (at 126.365 90.805))
+  (junction (at 111.125 121.285) (diameter 0) (color 0 0 0 0)
+  )
   (no_connect (at 126.365 111.125))
   (no_connect (at 126.365 103.505))
   (no_connect (at 126.365 95.885))
-  (no_connect (at 126.365 108.585))
-  (no_connect (at 126.365 93.345))
   (no_connect (at 95.885 100.965))
   (no_connect (at 126.365 98.425))
+  (wire (pts (xy 111.125 121.285) (xy 111.125 122.555))
+    (stroke (width 0) (type default))
+  )
   (wire (pts (xy 102.87 67.945) (xy 111.125 67.945))
     (stroke (width 0) (type default))
   )
+  (wire (pts (xy 126.365 108.585) (xy 129.54 108.585))
+    (stroke (width 0) (type default))
+  )
   (wire (pts (xy 186.69 118.745) (xy 194.31 118.745))
     (stroke (width 0) (type default))
@@
     (stroke (width 0) (type default))
   )
+  (wire (pts (xy 81.915 88.9) (xy 81.915 95.885))
+    (stroke (width 0) (type default))
+  )
   (wire (pts (xy 194.31 118.745) (xy 194.31 121.285))
     (stroke (width 0) (type default))
@@
     (stroke (width 0) (type default))
   )
+  (wire (pts (xy 81.915 81.28) (xy 81.915 67.945))
+    (stroke (width 0) (type default))
+  )
   (wire (pts (xy 194.31 136.525) (xy 204.47 136.525))
     (stroke (width 0) (type default))
@@
     (stroke (width 0) (type default))
   )
+  (wire (pts (xy 141.605 80.645) (xy 141.605 67.945))
+    (stroke (width 0) (type default))
+  )
   (wire (pts (xy 204.47 118.745) (xy 194.31 118.745))
     (stroke (width 0) (type default))
   )
+  (wire (pts (xy 129.54 121.285) (xy 111.125 121.285))
+    (stroke (width 0) (type default))
+  )
   (wire (pts (xy 185.42 65.405) (xy 185.42 70.485))
     (stroke (width 0) (type default))
   )
+  (wire (pts (xy 141.605 93.345) (xy 126.365 93.345))
+    (stroke (width 0) (type default))
+  )
   (wire (pts (xy 140.97 106.045) (xy 142.24 106.045))
     (stroke (width 0) (type default))
@@
     (stroke (width 0) (type default))
   )
+  (wire (pts (xy 129.54 108.585) (xy 129.54 110.49))
+    (stroke (width 0) (type default))
+  )
   (wire (pts (xy 171.45 70.485) (xy 180.34 70.485))
     (stroke (width 0) (type default))
@@
     (stroke (width 0) (type default))
   )
-  (wire (pts (xy 111.125 116.205) (xy 111.125 118.11))
+  (wire (pts (xy 111.125 116.205) (xy 111.125 121.285))
     (stroke (width 0) (type default))
   )
@@
     (stroke (width 0) (type default))
   )
+  (wire (pts (xy 141.605 88.265) (xy 141.605 93.345))
+    (stroke (width 0) (type default))
+  )
   (wire (pts (xy 90.17 111.125) (xy 95.885 111.125))
     (stroke (width 0) (type default))
   )
-  (wire (pts (xy 90.805 95.885) (xy 95.885 95.885))
+  (wire (pts (xy 81.915 95.885) (xy 95.885 95.885))
     (stroke (width 0) (type default))
   )
@@
     (stroke (width 0) (type default))
   )
+  (wire (pts (xy 135.255 90.805) (xy 126.365 90.805))
+    (stroke (width 0) (type default))
+  )
   (wire (pts (xy 194.31 114.935) (xy 194.31 118.745))
     (stroke (width 0) (type default))
@@
     (stroke (width 0) (type default))
   )
+  (wire (pts (xy 81.915 67.945) (xy 97.79 67.945))
+    (stroke (width 0) (type default))
+  )
   (wire (pts (xy 180.34 65.405) (xy 180.34 70.485))
     (stroke (width 0) (type default))
@@
     (stroke (width 0) (type default))
   )
+  (wire (pts (xy 129.54 118.11) (xy 129.54 121.285))
+    (stroke (width 0) (type default))
+  )
   (wire (pts (xy 133.35 106.045) (xy 126.365 106.045))
+    (stroke (width 0) (type default))
+  )
+  (wire (pts (xy 141.605 67.945) (xy 111.125 67.945))
     (stroke (width 0) (type default))
   )
@@
     (effects (font (size 1.27 1.27)) (justify left bottom))
   )
+  (label "BOOT" (at 135.255 90.805 180) (fields_autoplaced)
+    (effects (font (size 1.27 1.27)) (justify right bottom))
+  )
   (label "BOOT" (at 163.83 118.745 0) (fields_autoplaced)
     (effects (font (size 1.27 1.27)) (justify left bottom))
@@
   )
   (label "RST" (at 190.5 70.485 90) (fields_autoplaced)
-    (effects (font (size 1.27 1.27)) (justify left bottom))
-  )
-  (label "BOOT" (at 90.805 95.885 0) (fields_autoplaced)
     (effects (font (size 1.27 1.27)) (justify left bottom))
   )
@@
     )
   )
-  (symbol (lib_name "GND_3") (lib_id "power:GND") (at 111.125 118.11 0) (unit 1)
+  (symbol (lib_name "GND_3") (lib_id "power:GND") (at 111.125 122.555 0) (unit 1)
     (in_bom yes) (on_board yes) (dnp no) (fields_autoplaced)
-    (property "Reference" "#PWR031" (at 111.125 124.46 0)
-      (effects (font (size 1.27 1.27)) hide)
-    )
-    (property "Value" "GND" (at 111.125 123.19 0)
+    (property "Reference" "#PWR031" (at 111.125 128.905 0)
+      (effects (font (size 1.27 1.27)) hide)
+    )
+    (property "Value" "GND" (at 111.125 127.635 0)
       (effects (font (size 1.27 1.27)))
     )
-    (property "Footprint" "" (at 111.125 118.11 0)
-      (effects (font (size 1.27 1.27)) hide)
-    )
-    (property "Datasheet" "" (at 111.125 118.11 0)
+    (property "Footprint" "" (at 111.125 122.555 0)
+      (effects (font (size 1.27 1.27)) hide)
+    )
+    (property "Datasheet" "" (at 111.125 122.555 0)
       (effects (font (size 1.27 1.27)) hide)
     )
@@
     )
   )
+  (symbol (lib_id "Device:R") (at 141.605 84.455 0) (mirror x) (unit 1)
+    (in_bom yes) (on_board yes) (dnp no)
+    (property "Reference" "R51" (at 144.145 82.55 90)
+      (effects (font (size 1.27 1.27)) (justify left))
+    )
+    (property "Value" "10k" (at 139.065 83.185 90)
+      (effects (font (size 1.27 1.27)) (justify left))
+    )
+    (property "Footprint" "IVS_FOOTPRINTS:R_0603" (at 139.827 84.455 90)
+      (effects (font (size 1.27 1.27)) hide)
+    )
+    (property "Datasheet" "~" (at 141.605 84.455 0)
+      (effects (font (size 1.27 1.27)) hide)
+    )
+    (pin "1")
+    (pin "2")
+    (instances
+      (project "DLAnhDan_BoardTruyenDuLieu"
+        (path "/a9565029-c1f4-4226-96c5-abe75b48376f/e1e44dd4-10ee-4582-93a6-e8839f1980ca"
+          (reference "R51") (unit 1)
+        )
+      )
+      (project "DO_AN_DKTD"
+        (path "/fe9c1bbb-8428-4aad-931e-ea95c4d011b3/514f7f67-6c84-4d42-8fe7-76f8a193466f"
+          (reference "R34") (unit 1)
+        )
+      )
+    )
+  )
   (symbol (lib_name "GND_1") (lib_id "power:GND") (at 185.42 140.335 0) (unit 1)
     (in_bom yes) (on_board yes) (dnp no) (fields_autoplaced)
@@
     )
   )
+  (symbol (lib_id "Device:R") (at 129.54 114.3 0) (mirror x) (unit 1)
+    (in_bom yes) (on_board yes) (dnp no)
+    (property "Reference" "R51" (at 132.08 112.395 90)
+      (effects (font (size 1.27 1.27)) (justify left))
+    )
+    (property "Value" "10k" (at 127 113.03 90)
+      (effects (font (size 1.27 1.27)) (justify left))
+    )
+    (property "Footprint" "IVS_FOOTPRINTS:R_0603" (at 127.762 114.3 90)
+      (effects (font (size 1.27 1.27)) hide)
+    )
+    (property "Datasheet" "~" (at 129.54 114.3 0)
+      (effects (font (size 1.27 1.27)) hide)
+    )
+    (pin "1")
+    (pin "2")
+    (instances
+      (project "DLAnhDan_BoardTruyenDuLieu"
+        (path "/a9565029-c1f4-4226-96c5-abe75b48376f/e1e44dd4-10ee-4582-93a6-e8839f1980ca"
+          (reference "R51") (unit 1)
+        )
+      )
+      (project "DO_AN_DKTD"
+        (path "/fe9c1bbb-8428-4aad-931e-ea95c4d011b3/514f7f67-6c84-4d42-8fe7-76f8a193466f"
+          (reference "R35") (unit 1)
+        )
+      )
+    )
+  )
   (symbol (lib_name "GND_2") (lib_id "power:GND") (at 193.04 71.755 0) (unit 1)
     (in_bom yes) (on_board yes) (dnp no) (fields_autoplaced)
@@
         )
       )
+    )
+  )
+  (symbol (lib_id "Device:R") (at 81.915 85.09 0) (mirror x) (unit 1)
+    (in_bom yes) (on_board yes) (dnp no)
+    (property "Reference" "R51" (at 84.455 83.185 90)
+      (effects (font (size 1.27 1.27)) (justify left))
+    )
+    (property "Value" "10k" (at 79.375 83.82 90)
+      (effects (font (size 1.27 1.27)) (justify left))
+    )
+    (property "Footprint" "IVS_FOOTPRINTS:R_0603" (at 80.137 85.09 90)
+      (effects (font (size 1.27 1.27)) hide)
+    )
+    (property "Datasheet" "~" (at 81.915 85.09 0)
+      (effects (font (size 1.27 1.27)) hide)
+    )
+    (pin "1")
+    (pin "2")
+    (instances
+      (project "DLAnhDan_BoardTruyenDuLieu"
+        (path "/a9565029-c1f4-4226-96c5-abe75b48376f/e1e44dd4-10ee-4582-93a6-e8839f1980ca"
+          (reference "R51") (unit 1)
+        )
+      )
+      (project "DO_AN_DKTD"
+        (path "/fe9c1bbb-8428-4aad-931e-ea95c4d011b3/514f7f67-6c84-4d42-8fe7-76f8a193466f"
+          (reference "R33") (unit 1)
+        )
+      )
