File: DO_AN_DKTD/DO_AN_DKTD.kicad_sch (KiCad schematic)
At the start: 59 parts, among them J1 Conn_01x03, J2 Conn_01x02, J3 Conn_01x07, J4 Conn_01x04, J5 Conn_01x02, Q1 NPN, Q2 NPN, Q3 NPN, Q4 NPN, SW2 RotaryEncoder_Switch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

Commit message: code update
Parts:
- added R30, R31: 4k7, IVS_FOOTPRINTS:R0603, symbol Device:R
Connections:
- net +3V3: now also R30.1, R31.1
- net SCL: now also R30.2
- net SDA: now also R31.2
Changed lines of the file:
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@@
   (junction (at 33.02 26.035) (diameter 0) (color 0 0 0 0)
+  )
+  (junction (at 190.5 158.75) (diameter 0) (color 0 0 0 0)
   )
   (junction (at 114.3 36.195) (diameter 0) (color 0 0 0 0)
@@
     (stroke (width 0) (type default))
   )
-  (wire (pts (xy 200.025 168.91) (xy 208.28 168.91))
-    (stroke (width 0) (type default))
-  )
   (wire (pts (xy 266.7 61.595) (xy 267.97 61.595))
     (stroke (width 0) (type default))
@@
     (stroke (width 0) (type default))
   )
+  (wire (pts (xy 194.31 158.75) (xy 190.5 158.75))
+    (stroke (width 0) (type default))
+  )
   (wire (pts (xy 297.815 56.515) (xy 290.83 56.515))
     (stroke (width 0) (type default))
   )
+  (wire (pts (xy 190.5 158.75) (xy 186.055 158.75))
+    (stroke (width 0) (type default))
+  )
   (wire (pts (xy 283.21 64.135) (xy 270.51 64.135))
     (stroke (width 0) (type default))
@@
     (stroke (width 0) (type default))
   )
+  (wire (pts (xy 186.055 171.45) (xy 208.28 171.45))
+    (stroke (width 0) (type default))
+  )
   (wire (pts (xy 74.93 182.88) (xy 69.215 182.88))
     (stroke (width 0) (type default))
@@
     (stroke (width 0) (type default))
   )
+  (wire (pts (xy 190.5 157.48) (xy 190.5 158.75))
+    (stroke (width 0) (type default))
+  )
   (wire (pts (xy 200.025 43.815) (xy 200.025 51.435))
     (stroke (width 0) (type default))
@@
     (stroke (width 0) (type default))
   )
+  (wire (pts (xy 194.31 168.91) (xy 208.28 168.91))
+    (stroke (width 0) (type default))
+  )
   (wire (pts (xy 57.15 205.74) (xy 45.72 205.74))
     (stroke (width 0) (type default))
@@
     (stroke (width 0) (type default))
   )
+  (wire (pts (xy 186.055 158.75) (xy 186.055 161.29))
+    (stroke (width 0) (type default))
+  )
   (wire (pts (xy 49.53 142.875) (xy 49.53 153.035))
     (stroke (width 0) (type default))
@@
     (stroke (width 0) (type default))
   )
+  (wire (pts (xy 194.31 161.29) (xy 194.31 158.75))
+    (stroke (width 0) (type default))
+  )
   (wire (pts (xy 102.235 84.455) (xy 91.44 84.455))
     (stroke (width 0) (type default))
@@
     (stroke (width 0) (type default))
   )
-  (wire (pts (xy 200.025 171.45) (xy 208.28 171.45))
-    (stroke (width 0) (type default))
-  )
   (wire (pts (xy 358.14 80.645) (xy 358.14 92.71))
     (stroke (width 0) (type default))
@@
   )
   (wire (pts (xy 126.365 33.02) (xy 126.365 36.195))
+    (stroke (width 0) (type default))
+  )
+  (wire (pts (xy 186.055 168.91) (xy 186.055 171.45))
     (stroke (width 0) (type default))
   )
@@
     )
   )
+  (symbol (lib_id "Device:R") (at 186.055 165.1 0) (mirror y) (unit 1)
+    (in_bom yes) (on_board yes) (dnp no) (fields_autoplaced)
+    (property "Reference" "R31" (at 183.515 164.465 0)
+      (effects (font (size 1.27 1.27)) (justify left))
+    )
+    (property "Value" "4k7" (at 183.515 167.005 0)
+      (effects (font (size 1.27 1.27)) (justify left))
+    )
+    (property "Footprint" "IVS_FOOTPRINTS:R0603" (at 187.833 165.1 90)
+      (effects (font (size 1.27 1.27)) hide)
+    )
+    (property "Datasheet" "~" (at 186.055 165.1 0)
+      (effects (font (size 1.27 1.27)) hide)
+    )
+    (pin "1")
+    (pin "2")
+    (instances
+      (project "DO_AN_DKTD"
+        (path "/fe9c1bbb-8428-4aad-931e-ea95c4d011b3"
+          (reference "R31") (unit 1)
+        )
+      )
+    )
+  )
   (symbol (lib_id "Device:C") (at 74.93 199.39 0) (mirror y) (unit 1)
     (in_bom yes) (on_board yes) (dnp no) (fields_autoplaced)
@@
         (path "/fe9c1bbb-8428-4aad-931e-ea95c4d011b3"
           (reference "R7") (unit 1)
+        )
+      )
+    )
+  )
+  (symbol (lib_id "power:+3V3") (at 190.5 157.48 0) (unit 1)
+    (in_bom yes) (on_board yes) (dnp no) (fields_autoplaced)
+    (property "Reference" "#PWR010" (at 190.5 161.29 0)
+      (effects (font (size 1.27 1.27)) hide)
+    )
+    (property "Value" "+3V3" (at 190.5 153.67 0)
+      (effects (font (size 1.27 1.27)))
+    )
+    (property "Footprint" "" (at 190.5 157.48 0)
+      (effects (font (size 1.27 1.27)) hide)
+    )
+    (property "Datasheet" "" (at 190.5 157.48 0)
+      (effects (font (size 1.27 1.27)) hide)
+    )
+    (pin "1")
+    (instances
+      (project "DO_AN_DKTD"
+        (path "/fe9c1bbb-8428-4aad-931e-ea95c4d011b3"
+          (reference "#PWR010") (unit 1)
         )
       )
@@
         )
       )
+    )
+  )
+  (symbol (lib_id "Device:R") (at 194.31 165.1 0) (mirror y) (unit 1)
+    (in_bom yes) (on_board yes) (dnp no) (fields_autoplaced)
+    (property "Reference" "R30" (at 191.77 164.465 0)
+      (effects (font (size 1.27 1.27)) (justify left))
+    )
+    (property "Value" "4k7" (at 191.77 167.005 0)
+      (effects (font (size 1.27 1.27)) (justify left))
+    )
+    (property "Footprint" "IVS_FOOTPRINTS:R0603" (at 196.088 165.1 90)
+      (effects (font (size 1.27 1.27)) hide)
+    )
+    (property "Datasheet" "~" (at 194.31 165.1 0)
+      (effects (font (size 1.27 1.27)) hide)
+    )
+    (pin "1")
+    (pin "2")
+    (instances
+      (project "DO_AN_DKTD"
+        (path "/fe9c1bbb-8428-4aad-931e-ea95c4d011b3"
+          (reference "R30") (unit 1)
+        )
+      )

Commit message: completed layout PCB Ver 1.0
Parts:
- removed C1, C4, C9: 100nF, IVS_FOOTPRINTS:C_0603, symbol Device:C
- removed C2, C3: 1uF, IVS_FOOTPRINTS:C_0603, symbol Device:C
- removed C5: 50nF, IVS_FOOTPRINTS:C_0603, symbol Device:C
- removed C6, C7: 10nF, IVS_FOOTPRINTS:C_0603, symbol Device:C
- removed C8: 10uF, IVS_FOOTPRINTS:C_0603, symbol Device:C
- removed D1: TRIAC, IVS_FOOTPRINTS:TO-220-3_Vertical, symbol IVS_SYMBOLS:Triac
- removed D2: MB10F, IVS_FOOTPRINTS:Bridge_MB10F-13, symbol Device:D_Bridge_+A-A
- removed D3: 1N4148, IVS_FOOTPRINTS:D_SOD323, symbol IVS_SYMBOLS:D_Diode
- removed F1: Fuse, IVS_FOOTPRINTS:Fuse_BLX-A-P22.4mm, symbol IVS_SYMBOLS:Fuse
- removed F2: Fuse, IVS_FOOTPRINTS:Fuse_1812_4532Metric, symbol IVS_SYMBOLS:Fuse
- removed J1: Conn_01x03, IVS_FOOTPRINTS:Conn_XH-P2.54mm-3P, symbol Connector_Generic:Conn_01x03
- removed J2, J5: Conn_01x02, IVS_FOOTPRINTS:KF128-5.0-2P, symbol Connector_Generic:Conn_01x02
- removed J3: Conn_01x07, IVS_FOOTPRINTS:Conn_XH-P2.54mm-7P, symbol Connector_Generic:Conn_01x07
- removed J4: Conn_01x04, IVS_FOOTPRINTS:Conn_XH-P2.54mm-4P, symbol Connector_Generic:Conn_01x04
- removed LE1: 5631AS, IVS_FOOTPRINTS:7Segment_4led_CC_38x19, symbol IVS_SYMBOLS:7seg_5631AS
- removed Q1, Q2, Q3, Q4: NPN, IVS_FOOTPRINTS:SOT23-3, symbol IVS_SYMBOLS:NPN
- removed R1, R15, R16, R17, R18, R2, R3, R30, R31: 4k7, IVS_FOOTPRINTS:R0603, symbol Device:R
- removed R10, R11, R25, R27, R4, R5, R6, R7, R8, R9: 1k, IVS_FOOTPRINTS:R0603, symbol Device:R
- removed R12, R13, R14: 2k, IVS_FOOTPRINTS:R0603, symbol Device:R
- removed R19: 360, IVS_FOOTPRINTS:R0805, symbol Device:R
- removed R20: 470, IVS_FOOTPRINTS:R0603, symbol Device:R
- removed R21: 39, IVS_FOOTPRINTS:R0603, symbol Device:R
- removed R22: 360, IVS_FOOTPRINTS:R0603, symbol Device:R
- removed R23, R24: 180k, IVS_FOOTPRINTS:R0603, symbol Device:R
- removed R26: 22k, IVS_FOOTPRINTS:R0603, symbol Device:R
- removed R28, R29: 0R, IVS_FOOTPRINTS:R0805, symbol Device:R
- removed SW2: RotaryEncoder_Switch, IVS_FOOTPRINTS:RotaryEncoder_Alps_EC11E-Switch_Vertical_H20mm, symbol IVS_SYMBOLS:RotaryEncoder_Switch
- removed U1: AMS1117, IVS_FOOTPRINTS:SOT233, symbol IVS_SYMBOLS:AMS1117
- removed U2: 74HC595, IVS_FOOTPRINTS:SOIC-16W_5.3x10.2mm_P1.27mm, symbol 74xx:74HC595
- removed U3: MOC3020M, IVS_FOOTPRINTS:DIL06-E, symbol Relay_SolidState:MOC3020M
- removed U4: PC817, IVS_FOOTPRINTS:OPTO_SOT254P975X400-4N, symbol Isolator:EL817
- removed U5: DevKitSTM32, IVS_FOOTPRINTS:DevKitSTM32, symbol IVS_SYMBOLS:DevKitSTM32
Connections:
- no-connect marks 24 -> 0
Other:
- added sheet ESP (ESP.kicad_sch)
- added sheet POWER (POWER.kicad_sch)
- added sheet Peripheral (Peripheral.kicad_sch)
- added sheet STM32 (STM32.kicad_sch)
- note removed: "I2C"
- note removed: "POWER"
- note removed: "UART"
