File: DO_AN_DKTD/POWER.kicad_sch (KiCad schematic)
At the start: 24 parts, among them J2 Jack-DC, J3 Conn_01x07, Q10 P_Mosfet, U1 AMS1117, U1 XL1509

Commit message: commit to change branch
Other:
- moved on the sheet: C1, C2, C24, C26, C27, C3, C4, D6, D7, D8, F2, J2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

Commit message: complete code DO_AN_MON
Parts:
- removed D7: D_Schottky, IVS_FOOTPRINTS:D_SOD323, symbol IVS_SYMBOLS:D_Schottky
- added Z1: D_Zener, symbol IVS_SYMBOLS:D_Zener
Connections:
- net VDC: now also Z1.2
- net at C26.1, Q10.1 (G), R32.1: now also Z1.1
Changed lines of the file:
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@@
+    )
+  )
+  (symbol (lib_id "IVS_SYMBOLS:D_Zener") (at 113.665 63.5 270) (unit 1)
+    (in_bom yes) (on_board yes) (dnp no)
+    (property "Reference" "Z1" (at 118.11 63.5 90)
+      (effects (font (size 1.27 1.27)) (justify left))
+    )
+    (property "Value" "D_Zener" (at 116.205 66.04 90)
+      (effects (font (size 1.27 1.27)) (justify left))
+    )
+    (property "Footprint" "" (at 113.665 63.5 0)
+      (effects (font (size 1.27 1.27)) hide)
+    )
+    (property "Datasheet" "" (at 113.665 63.5 0)
+      (effects (font (size 1.27 1.27)) hide)
+    )
+    (pin "1")
+    (pin "2")
+    (instances
+      (project "DO_AN_DKTD"
+        (path "/fe9c1bbb-8428-4aad-931e-ea95c4d011b3/24a20ba6-d689-4def-9a51-4ba12b1afb4b"
+          (reference "Z1") (unit 1)
+        )
+      )
     )
   )
@@
         )
       )
-    )
-  )
-  (symbol (lib_id "IVS_SYMBOLS:D_Schottky") (at 113.665 63.5 270) (unit 1)
-    (in_bom yes) (on_board yes) (dnp no) (fields_autoplaced)
-    (property "Reference" "D7" (at 116.205 63.8175 90)
-      (effects (font (size 1.27 1.27)) (justify left))
-    )
-    (property "Value" "D_Schottky" (at 116.205 66.3575 90)
-      (effects (font (size 1.27 1.27)) (justify left))
-    )
-    (property "Footprint" "IVS_FOOTPRINTS:D_SOD323" (at 113.665 63.5 0)
-      (effects (font (size 1.27 1.27)) hide)
-    )
-    (property "Datasheet" "" (at 113.665 63.5 0)
-      (effects (font (size 1.27 1.27)) hide)
-    )
-    (pin "1")
-    (pin "2")
-    (instances
-      (project "DO_AN_DKTD"
-        (path "/fe9c1bbb-8428-4aad-931e-ea95c4d011b3/24a20ba6-d689-4def-9a51-4ba12b1afb4b"
-          (reference "D7") (unit 1)
-        )
-      )
